File: RH006/RH006.1/RH006.1.sch (EAGLE design)
At the start: 39 parts, among them CN1 USB, CN4 FTDI, Q2 BSS138, Q3 BSS138, U1 ATMega-328, U3 MCP1703CB, X1 16 MHz

Commit message: Prepare board 6 for production, version 1 finished
Connections:
- removed net VCC: Q2.G, Q3.G, R3.1, R5.1
- net 3.3V: now also Q2.G, Q3.G, R3.1, R5.1
Changed lines of the file:
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@@
 <label x="210.82" y="53.34" size="1.778" layer="95"/>
+</segment>
+<segment>
+<wire x1="64.77" y1="27.94" x2="64.77" y2="30.48" width="0.1524" layer="91"/>
+<wire x1="72.39" y1="22.86" x2="72.39" y2="30.48" width="0.1524" layer="91"/>
+<wire x1="72.39" y1="30.48" x2="64.77" y2="30.48" width="0.1524" layer="91"/>
+<junction x="64.77" y="30.48"/>
+<pinref part="R3" gate="G$1" pin="1"/>
+<pinref part="Q2" gate="G$1" pin="G"/>
+<pinref part="P+2" gate="1" pin="VCC"/>
+<wire x1="64.77" y1="35.56" x2="64.77" y2="30.48" width="0.1524" layer="91"/>
+</segment>
+<segment>
+<wire x1="113.03" y1="27.94" x2="113.03" y2="30.48" width="0.1524" layer="91"/>
+<wire x1="120.65" y1="22.86" x2="120.65" y2="30.48" width="0.1524" layer="91"/>
+<wire x1="120.65" y1="30.48" x2="113.03" y2="30.48" width="0.1524" layer="91"/>
+<junction x="113.03" y="30.48"/>
+<pinref part="R5" gate="G$1" pin="1"/>
+<pinref part="Q3" gate="G$1" pin="G"/>
+<pinref part="P+3" gate="1" pin="VCC"/>
+<wire x1="113.03" y1="35.56" x2="113.03" y2="30.48" width="0.1524" layer="91"/>
 </segment>
 </net>
@@
 </segment>
 </net>
-<net name="VCC" class="0">
-<segment>
-<wire x1="64.77" y1="27.94" x2="64.77" y2="30.48" width="0.1524" layer="91"/>
-<wire x1="72.39" y1="22.86" x2="72.39" y2="30.48" width="0.1524" layer="91"/>
-<wire x1="72.39" y1="30.48" x2="64.77" y2="30.48" width="0.1524" layer="91"/>
-<junction x="64.77" y="30.48"/>
-<pinref part="R3" gate="G$1" pin="1"/>
-<pinref part="Q2" gate="G$1" pin="G"/>
-<pinref part="P+2" gate="1" pin="VCC"/>
-<wire x1="64.77" y1="35.56" x2="64.77" y2="30.48" width="0.1524" layer="91"/>
-</segment>
-<segment>
-<wire x1="113.03" y1="27.94" x2="113.03" y2="30.48" width="0.1524" layer="91"/>
-<wire x1="120.65" y1="22.86" x2="120.65" y2="30.48" width="0.1524" layer="91"/>
-<wire x1="120.65" y1="30.48" x2="113.03" y2="30.48" width="0.1524" layer="91"/>
-<junction x="113.03" y="30.48"/>
-<pinref part="R5" gate="G$1" pin="1"/>
-<pinref part="Q3" gate="G$1" pin="G"/>
-<pinref part="P+3" gate="1" pin="VCC"/>
-<wire x1="113.03" y1="35.56" x2="113.03" y2="30.48" width="0.1524" layer="91"/>
-</segment>
-</net>
