File: RH009/RH009.1/RH009.1.brd (EAGLE design)
At the start: 49.5 x 49.5 mm, 23 parts, among them Q2 BSS138, Q3 BSS138

Commit message: Minor fixes
Connections:
- removed net PWR: A3.2, JP3.13
- net VBUS: now also A3.2, JP3.13
Routing:
- net VBUS: track 7.59 -> 118.1 mm, vias 0 -> 1
- net PWR: track 79.2 -> 0.00 mm
Changed lines of the file:
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@@
 </element>
 <element name="U2" library="microbuilder" package="SOP28_300MIL" value="" x="24.765" y="24.765" smashed="yes" rot="MR0">
-<attribute name="NAME" x="32.385" y="26.035" size="0.8128" layer="26" ratio="18" rot="MR0"/>
+<attribute name="NAME" x="35.941" y="27.559" size="0.8128" layer="26" ratio="18" rot="MR0"/>
 <attribute name="VALUE" x="32.385" y="24.765" size="0.4064" layer="28" ratio="10" rot="MR0"/>
 </element>
@@
 <signal name="D10_SS">
 <contactref element="JP5" pad="8"/>
-</signal>
-<signal name="PWR" class="1">
-<contactref element="JP3" pad="13"/>
-<contactref element="A3" pad="2"/>
-<wire x1="45.72" y1="40.4622" x2="45.72" y2="39.878" width="0.381" layer="16"/>
-<wire x1="46.4058" y1="41.148" x2="45.72" y2="40.4622" width="0.381" layer="16"/>
-<wire x1="48.006" y1="41.148" x2="46.4058" y2="41.148" width="0.381" layer="16"/>
-<wire x1="48.9204" y1="40.2336" x2="48.006" y2="41.148" width="0.381" layer="16"/>
-<wire x1="48.9204" y1="8.6868" x2="48.9204" y2="40.2336" width="0.381" layer="16"/>
-<wire x1="42.7482" y1="2.5146" x2="48.9204" y2="8.6868" width="0.381" layer="16"/>
-<wire x1="42.7482" y1="0.8001" x2="42.7482" y2="2.5146" width="0.381" layer="16"/>
-<wire x1="42.4053" y1="0.4572" x2="42.7482" y2="0.8001" width="0.381" layer="16"/>
-<wire x1="12.1158" y1="0.4572" x2="42.4053" y2="0.4572" width="0.381" layer="16"/>
-<wire x1="10.7442" y1="1.8288" x2="12.1158" y2="0.4572" width="0.381" layer="16"/>
-<wire x1="10.7442" y1="1.8288" x2="10.795" y2="1.905" width="0.381" layer="16"/>
 </signal>
 <signal name="D9">
@@
 <wire x1="7.0866" y1="27.2034" x2="5.9436" y2="28.3464" width="0.381" layer="16"/>
 <wire x1="7.0866" y1="27.0891" x2="7.0866" y2="27.2034" width="0.381" layer="16"/>
-<wire x1="7.5438" y1="26.6319" x2="7.0866" y2="27.0891" width="0.381" layer="16"/>
+<wire x1="7.5438" y1="26.6319" x2="7.2009" y2="26.9748" width="0.381" layer="16"/>
+<wire x1="7.2009" y1="26.9748" x2="7.0866" y2="27.0891" width="0.381" layer="16"/>
 <wire x1="10.1727" y1="26.6319" x2="7.5438" y2="26.6319" width="0.381" layer="16"/>
 <wire x1="11.8872" y1="28.3464" x2="10.1727" y2="26.6319" width="0.381" layer="16"/>
 <wire x1="5.9436" y1="28.3464" x2="5.842" y2="28.36" width="0.381" layer="16"/>
 <wire x1="11.8872" y1="28.3464" x2="11.938" y2="28.36" width="0.381" layer="16"/>
+<contactref element="JP3" pad="13"/>
+<contactref element="A3" pad="2"/>
+<wire x1="45.72" y1="40.4622" x2="45.72" y2="39.878" width="0.381" layer="16"/>
+<wire x1="46.4058" y1="41.148" x2="45.72" y2="40.4622" width="0.381" layer="16"/>
+<wire x1="48.006" y1="41.148" x2="46.4058" y2="41.148" width="0.381" layer="16"/>
+<wire x1="48.9204" y1="40.2336" x2="48.006" y2="41.148" width="0.381" layer="16"/>
+<wire x1="48.9204" y1="8.6868" x2="48.9204" y2="40.2336" width="0.381" layer="16"/>
+<wire x1="42.7482" y1="2.5146" x2="48.9204" y2="8.6868" width="0.381" layer="16"/>
+<wire x1="42.7482" y1="0.8001" x2="42.7482" y2="2.5146" width="0.381" layer="16"/>
+<wire x1="42.4053" y1="0.4572" x2="42.7482" y2="0.8001" width="0.381" layer="16"/>
+<wire x1="12.1158" y1="0.4572" x2="42.4053" y2="0.4572" width="0.381" layer="16"/>
+<wire x1="10.7442" y1="1.8288" x2="12.1158" y2="0.4572" width="0.381" layer="16"/>
+<wire x1="7.0866" y1="26.7462" x2="7.0866" y2="26.8605" width="0.381" layer="16"/>
+<wire x1="7.0866" y1="3.3147" x2="7.0866" y2="26.7462" width="0.381" layer="1"/>
+<wire x1="6.7437" y1="2.9718" x2="7.0866" y2="3.3147" width="0.381" layer="1"/>
+<wire x1="6.7437" y1="0.8001" x2="6.7437" y2="2.9718" width="0.381" layer="1"/>
+<wire x1="7.0866" y1="0.4572" x2="6.7437" y2="0.8001" width="0.381" layer="1"/>
+<wire x1="9.3726" y1="0.4572" x2="7.0866" y2="0.4572" width="0.381" layer="1"/>
+<wire x1="10.7442" y1="1.8288" x2="9.3726" y2="0.4572" width="0.381" layer="1"/>
+<wire x1="7.0866" y1="26.8605" x2="7.2009" y2="26.9748" width="0.381" layer="16"/>
+<wire x1="10.7442" y1="1.8288" x2="10.795" y2="1.905" width="0.381" layer="1"/>
+<wire x1="10.8585" y1="1.9431" x2="10.795" y2="1.905" width="0.381" layer="16"/>
+<wire x1="10.8585" y1="1.9431" x2="10.7442" y2="1.8288" width="0.381" layer="16"/>
+<via x="7.0866" y="26.7462" extent="1-16" drill="0.3048"/>
 </signal>
 <signal name="3.3V">

Commit message: Board 9.1 finished
Parts:
- moved U$3 10.7 mm to (46.6, 8.23)
Connections:
- removed net VCC: Q2.1, Q3.1, R3.1, R5.1
- net 3.3V: now also Q2.1, Q3.1, R3.1, R5.1
Routing:
- net 3.3V: track 63.0 -> 114.8 mm, vias 0 -> 4
- net VCC: track 19.8 -> 0.00 mm
Other:
- board text added: "3.3v"
- board text added: "3.3v i2c"
- board text added: "5v"
- board text added: "LED Power"
- board text added: "RH009.1 Mar 2015"
- board text removed: "3.3V"
- board text removed: "5V"
- board text removed: "5V I2C"
- board text removed: "RH009.1 Feb 2015"
Changed lines of the file:
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@@
 <wire x1="49.53" y1="46.355" x2="49.53" y2="3.175" width="0.0254" layer="20"/>
 <text x="1.27" y="38.9255" size="1.016" layer="25">RH009.1
-Feb 2015</text>
+Mar 2015</text>
 <text x="7.239" y="44.16425" size="1.016" layer="25">Matrix Shield
 Richard Hawthorn
@@
 <text x="35.3695" y="43.815" size="1.016" layer="25">MI</text>
 <text x="32.8295" y="43.815" size="1.016" layer="25">SK</text>
-<text x="29.9085" y="44.958" size="1.016" layer="25">A5</text>
-<text x="27.3685" y="44.958" size="1.016" layer="25">A4</text>
-<text x="24.8285" y="44.958" size="1.016" layer="25">A3</text>
-<text x="22.2885" y="44.958" size="1.016" layer="25">A2</text>
-<text x="29.6545" y="43.8785" size="0.8128" layer="25">SCL</text>
-<text x="27.1145" y="43.8785" size="0.8128" layer="25">SDA</text>
+<text x="30.1625" y="44.958" size="1.016" layer="25">A5</text>
+<text x="27.6225" y="44.958" size="1.016" layer="25">A4</text>
+<text x="25.0825" y="44.958" size="1.016" layer="25">A3</text>
+<text x="22.5425" y="44.958" size="1.016" layer="25">A2</text>
+<text x="29.9085" y="43.8785" size="0.8128" layer="25">SCL</text>
+<text x="27.3685" y="43.8785" size="0.8128" layer="25">SDA</text>
 <text x="9.906" y="3.683" size="0.762" layer="25">VIN</text>
 <text x="12.7" y="3.683" size="0.8128" layer="25">3.3</text>
@@
 <text x="40.894" y="3.683" size="1.016" layer="25">A1</text>
 <text x="7.112" y="3.683" size="0.762" layer="25">GND</text>
-<text x="43.18" y="39.116" size="1.27" layer="26" rot="MR0">5V</text>
-<text x="43.18" y="35.56" size="1.27" layer="26" rot="MR0">3.3V</text>
-<text x="43.688" y="29.464" size="1.27" layer="26" rot="MR0">5V I2C</text>
+<text x="43.18" y="39.116" size="1.27" layer="26" rot="MR0">5v</text>
+<text x="43.18" y="35.56" size="1.27" layer="26" rot="MR0">3.3v</text>
+<text x="43.688" y="29.464" size="1.27" layer="26" rot="MR0">3.3v i2c</text>
+<text x="43.18" y="41.402" size="1.016" layer="26" rot="MR0">LED Power</text>
 </plain>
 <attributes>
@@
 </autorouter>
 <elements>
-<element name="U$3" library="SparkFun-Aesthetics" package="OSHW-LOGO-S" value="" x="46.8249" y="18.8976" rot="MR90"/>
+<element name="U$3" library="SparkFun-Aesthetics" package="OSHW-LOGO-S" value="" x="46.5709" y="8.2296" rot="MR90"/>
 <element name="JP3" library="pinhead" package="1X14" value="" x="24.765" y="1.905" smashed="yes" rot="R180">
 <attribute name="VALUE" x="42.545" y="5.08" size="1.27" layer="27" rot="R180"/>
@@
 <wire x1="14.6304" y1="3.2004" x2="37.0332" y2="3.2004" width="0.3048" layer="16"/>
 <wire x1="13.335" y1="1.905" x2="14.6304" y2="3.2004" width="0.3048" layer="16"/>
+<contactref element="Q2" pad="1"/>
+<contactref element="R3" pad="1"/>
+<contactref element="Q3" pad="1"/>
+<contactref element="R5" pad="1"/>
+<wire x1="5.6007" y1="22.6314" x2="4.572" y2="22.6314" width="0.3048" layer="16"/>
+<wire x1="6.6294" y1="23.6601" x2="5.77215" y2="22.80285" width="0.3048" layer="16"/>
+<wire x1="5.77215" y1="22.80285" x2="5.6007" y2="22.6314" width="0.3048" layer="16"/>
+<wire x1="8.1153" y1="23.6601" x2="6.6294" y2="23.6601" width="0.3048" layer="16"/>
+<wire x1="8.8011" y1="22.9743" x2="8.1153" y2="23.6601" width="0.3048" layer="16"/>
+<wire x1="8.8011" y1="22.6314" x2="8.8011" y2="22.9743" width="0.3048" layer="16"/>
+<wire x1="8.8011" y1="22.6314" x2="8.824" y2="22.622" width="0.3048" layer="16"/>
+<wire x1="4.3434" y1="30.0609" x2="2.8575" y2="30.0609" width="0.3048" layer="16"/>
+<wire x1="5.2578" y1="30.9753" x2="4.3434" y2="30.0609" width="0.3048" layer="16"/>
+<wire x1="7.8867" y1="30.9753" x2="5.2578" y2="30.9753" width="0.3048" layer="16"/>
+<wire x1="8.8011" y1="30.0609" x2="7.8867" y2="30.9753" width="0.3048" layer="16"/>
+<wire x1="8.8011" y1="30.0609" x2="8.89" y2="30.06" width="0.3048" layer="16"/>
+<wire x1="4.4577" y1="30.0609" x2="4.4577" y2="29.845" width="0.3048" layer="16"/>
+<wire x1="4.4577" y1="29.845" x2="4.4577" y2="22.86" width="0.3048" layer="16"/>
+<wire x1="4.4577" y1="22.86" x2="4.4577" y2="22.7457" width="0.3048" layer="16"/>
+<wire x1="4.4577" y1="30.0609" x2="4.3434" y2="30.0609" width="0.3048" layer="16"/>
+<wire x1="4.445" y1="22.86" x2="4.4577" y2="22.86" width="0.3048" layer="16"/>
+<wire x1="5.715" y1="22.86" x2="4.4577" y2="22.86" width="0.3048" layer="16"/>
+<wire x1="4.445" y1="22.86" x2="4.506" y2="22.622" width="0.3048" layer="16"/>
+<wire x1="3.81" y1="30.48" x2="3.175" y2="30.48" width="0.3048" layer="16"/>
+<wire x1="4.445" y1="29.845" x2="3.81" y2="30.48" width="0.3048" layer="16"/>
+<wire x1="3.175" y1="30.48" x2="2.794" y2="30.06" width="0.3048" layer="16"/>
+<wire x1="4.445" y1="29.845" x2="4.4577" y2="29.845" width="0.3048" layer="16"/>
+<wire x1="5.715" y1="20.955" x2="5.715" y2="22.86" width="0.3048" layer="1"/>
+<wire x1="9.525" y1="20.955" x2="5.715" y2="20.955" width="0.3048" layer="16"/>
+<wire x1="9.525" y1="4.445" x2="9.525" y2="20.955" width="0.3048" layer="16"/>
+<wire x1="13.335" y1="4.445" x2="9.525" y2="4.445" width="0.3048" layer="1"/>
+<wire x1="13.335" y1="1.905" x2="13.335" y2="4.445" width="0.3048" layer="16"/>
+<wire x1="5.715" y1="22.86" x2="5.77215" y2="22.80285" width="0.3048" layer="16"/>
+<via x="5.715" y="22.86" extent="1-16" drill="0.3048"/>
+<via x="5.715" y="20.955" extent="1-16" drill="0.3048"/>
+<via x="9.525" y="4.445" extent="1-16" drill="0.3048"/>
+<via x="13.335" y="4.445" extent="1-16" drill="0.3048"/>
 </signal>
 <signal name="N$19">
@@
 <via x="10.8585" y="28.9179" extent="1-16" drill="0.3048"/>
 </signal>
-<signal name="VCC">
-<contactref element="Q2" pad="1"/>
-<contactref element="R3" pad="1"/>
-<contactref element="Q3" pad="1"/>
-<contactref element="R5" pad="1"/>
-<wire x1="5.6007" y1="22.6314" x2="4.572" y2="22.6314" width="0.3048" layer="16"/>
-<wire x1="6.6294" y1="23.6601" x2="5.6007" y2="22.6314" width="0.3048" layer="16"/>
-<wire x1="8.1153" y1="23.6601" x2="6.6294" y2="23.6601" width="0.3048" layer="16"/>
-<wire x1="8.8011" y1="22.9743" x2="8.1153" y2="23.6601" width="0.3048" layer="16"/>
-<wire x1="8.8011" y1="22.6314" x2="8.8011" y2="22.9743" width="0.3048" layer="16"/>
-<wire x1="4.572" y1="22.6314" x2="4.506" y2="22.622" width="0.3048" layer="16"/>
-<wire x1="8.8011" y1="22.6314" x2="8.824" y2="22.622" width="0.3048" layer="16"/>
-<wire x1="4.3434" y1="30.0609" x2="2.8575" y2="30.0609" width="0.3048" layer="16"/>
-<wire x1="5.2578" y1="30.9753" x2="4.3434" y2="30.0609" width="0.3048" layer="16"/>
-<wire x1="7.8867" y1="30.9753" x2="5.2578" y2="30.9753" width="0.3048" layer="16"/>
-<wire x1="8.8011" y1="30.0609" x2="7.8867" y2="30.9753" width="0.3048" layer="16"/>
-<wire x1="2.8575" y1="30.0609" x2="2.794" y2="30.06" width="0.3048" layer="16"/>
-<wire x1="8.8011" y1="30.0609" x2="8.89" y2="30.06" width="0.3048" layer="16"/>
-<wire x1="4.4577" y1="30.0609" x2="4.4577" y2="22.7457" width="0.3048" layer="16"/>
-<wire x1="4.4577" y1="22.7457" x2="4.506" y2="22.622" width="0.3048" layer="16"/>
-<wire x1="4.4577" y1="30.0609" x2="4.3434" y2="30.0609" width="0.3048" layer="16"/>
-</signal>
 <signal name="VLED" class="1">
